File: hardware/mouse/mouse.kicad_pcb (KiCad board)
At the start: 4 copper layers, 64 x 94 mm, 51 parts, among them J1 USB-C HRO TYPE-C-31-M-12, J10 Encoder: A / GND / B, J2 SWD: VDD / SWDIO / SWDCLK / G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, J3 Protected 1S 300mAh + 10k NTC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, J4 Charger status: GND / PGOOD /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, J5 BUTTON_LEFT contact, J6 BUTTON_RIGHT contact, J7 BUTTON_MIDDLE contact, J8 BUTTON_BACK contact, J9 BUTTON_FORWARD contact, SW1 PAIR TL3342, SW2 RESET TL3342, SW3 Power PCM12, U1 MDBT50Q-1MV2, U2 USBLC6-2SC6, U3 TLV70030DDCR, U4 PAW3395DM-T6QU, U5 TLV70019DDCR, U6 BQ24072RGTR, Y1 32.768kHz 12.5pF ABS07

Commit message: Route A1 prototype boards and build native firmware; bench validation pending
Parts:
- U6: footprint OpenMice:VQFN-16-1EP_3x3mm_P0.5mm_EP1.45x1.45mm -> OpenMice:BQ24072_RGT0016C
- moved R2 10.1 mm to (39.0, 9.00)
- moved U2 7.16 mm to (32.0, 11.5), turned to 90 degrees
- moved SW3 7.00 mm to (7.00, 56.0)
- moved J9 5.10 mm to (10.0, 43.0)
- moved J7 4.47 mm to (34.0, 22.0)
- moved R4 4.47 mm to (38.0, 56.0)
- moved C5 3.03 mm to (38.0, 11.0)
- moved J3 3.00 mm to (6.00, 50.0)
- moved R3 3.00 mm to (17.0, 84.0)
- moved C17 2.83 mm to (22.0, 15.0)
- moved J6 2.24 mm to (45.0, 23.0)
- moved J8 2.00 mm to (5.00, 37.0)
- moved R1 1.72 mm to (25.0, 9.00)
- turned J1 to 180 degrees
Connections:
- net BATTERY renamed /BATTERY
- net BATTERY_ADC renamed /BATTERY_ADC
- net BATTERY_NTC renamed /BATTERY_NTC
- net BUTTON_BACK renamed /BUTTON_BACK
- net BUTTON_FORWARD renamed /BUTTON_FORWARD
- net BUTTON_LEFT renamed /BUTTON_LEFT
- net BUTTON_MIDDLE renamed /BUTTON_MIDDLE
- net BUTTON_RIGHT renamed /BUTTON_RIGHT
- net CC1 renamed /CC1
- net CC2 renamed /CC2
- net CHARGER_ILIM renamed /CHARGER_ILIM
- net CHARGER_ISET renamed /CHARGER_ISET
- net CHARGER_TMR renamed /CHARGER_TMR
- net CHARGING renamed /CHARGING
- net ENCODER_A renamed /ENCODER_A
- net ENCODER_B renamed /ENCODER_B
- net GND renamed /GND
- net LF_XL1 renamed /LF_XL1
- net LF_XL2 renamed /LF_XL2
- net MCU_RESET renamed /MCU_RESET
- net PAIR renamed /PAIR
- net POWER_GOOD renamed /POWER_GOOD
- net SENSOR_IRQ renamed /SENSOR_IRQ
- net SENSOR_LED_P renamed /SENSOR_LED_P
- net SENSOR_NCS renamed /SENSOR_NCS
- net SENSOR_RESET renamed /SENSOR_RESET
- net SENSOR_VDDREG renamed /SENSOR_VDDREG
- net SPI_MISO renamed /SPI_MISO
- net SPI_MOSI renamed /SPI_MOSI
- net SPI_SCLK renamed /SPI_SCLK
- net SWDCLK renamed /SWDCLK
- net SWDIO renamed /SWDIO
- net SYSTEM renamed /SYSTEM
- net SYSTEM_ON renamed /SYSTEM_ON
- net USB_DM renamed /USB_DM
- net USB_DP renamed /USB_DP
- net USB_VBUS renamed /USB_VBUS
- net VDD_1V9 renamed /VDD_1V9
- net VDD_3V0 renamed /VDD_3V0
- J1 pad A8: (no net) -> unconnected-(J1-PadA8)
- J1 pad B8: (no net) -> unconnected-(J1-PadB8)
- SW3 pad 3: (no net) -> unconnected-(SW3-Pad3)
- U1 pad 10: (no net) -> unconnected-(U1-P0.29/AIN5-Pad10)
- U1 pad 11: (no net) -> unconnected-(U1-P0.02/AIN0-Pad11)
- U1 pad 12: (no net) -> unconnected-(U1-P0.31/AIN7-Pad12)
- U1 pad 13: (no net) -> unconnected-(U1-P0.28/AIN4-Pad13)
- U1 pad 14: (no net) -> unconnected-(U1-P0.30/AIN6-Pad14)
- U1 pad 21: (no net) -> unconnected-(U1-P0.05/AIN3-Pad21)
- U1 pad 22: (no net) -> unconnected-(U1-P0.06-Pad22)
- U1 pad 23: (no net) -> unconnected-(U1-TRACECLK/P0.07-Pad23)
- U1 pad 24: (no net) -> unconnected-(U1-P0.08-Pad24)
- U1 pad 25: (no net) -> unconnected-(U1-P1.08-Pad25)
- U1 pad 26: (no net) -> unconnected-(U1-TRACEDATA3/P1.09-Pad26)
- U1 pad 29: (no net) -> unconnected-(U1-TRACEDATA1/P0.12-Pad29)
- U1 pad 3: (no net) -> unconnected-(U1-P1.10-Pad3)
- U1 pad 31: (no net) -> unconnected-(U1-DCCH-Pad31)
- U1 pad 4: (no net) -> unconnected-(U1-P1.11-Pad4)
- U1 pad 42: (no net) -> unconnected-(U1-P0.19-Pad42)
- U1 pad 47: (no net) -> unconnected-(U1-TRACEDATA0/P1.00-Pad47)
- U1 pad 5: (no net) -> unconnected-(U1-P1.12-Pad5)
- U1 pad 50: (no net) -> unconnected-(U1-P1.02-Pad50)
- U1 pad 52: (no net) -> unconnected-(U1-P0.09/NFC1-Pad52)
- U1 pad 54: (no net) -> unconnected-(U1-P0.10/NFC2-Pad54)
- U1 pad 56: (no net) -> unconnected-(U1-P1.04-Pad56)
- U1 pad 57: (no net) -> unconnected-(U1-P1.06-Pad57)
- U1 pad 58: (no net) -> unconnected-(U1-P1.07-Pad58)
- U1 pad 59: (no net) -> unconnected-(U1-P1.05-Pad59)
- U1 pad 6: (no net) -> unconnected-(U1-P1.13-Pad6)
- U1 pad 60: (no net) -> unconnected-(U1-P1.03-Pad60)
- U1 pad 61: (no net) -> unconnected-(U1-P1.01-Pad61)
- U1 pad 7: (no net) -> unconnected-(U1-P1.14-Pad7)
- U1 pad 8: (no net) -> unconnected-(U1-P1.15-Pad8)
- U1 pad 9: (no net) -> unconnected-(U1-P0.03/AIN1-Pad9)
- U3 pad 4: (no net) -> unconnected-(U3-Pad4)
- U4 pad 1: (no net) -> unconnected-(U4-NC-Pad1)
- U4 pad 16: (no net) -> unconnected-(U4-NC-Pad16)
- U4 pad 2: (no net) -> unconnected-(U4-NC-Pad2)
- U4 pad 6: (no net) -> unconnected-(U4-NC-Pad6)
- U5 pad 4: (no net) -> unconnected-(U5-Pad4)
Routing:
- net /GND: track 0.00 -> 409.6 mm, vias 0 -> 18
- net /VDD_3V0: track 0.00 -> 187.3 mm, vias 0 -> 5
- net /USB_VBUS: track 0.00 -> 120.3 mm, vias 0 -> 5
- net /USB_DP: track 0.00 -> 109.6 mm, vias 0 -> 2
- net /USB_DM: track 0.00 -> 108.7 mm, vias 0 -> 2
- net /ENCODER_A: track 0.00 -> 80.5 mm, vias 0 -> 2
- net /BUTTON_RIGHT: track 0.00 -> 80.1 mm, vias 0 -> 1
- net /BUTTON_MIDDLE: track 0.00 -> 74.4 mm, vias 0 -> 3
- net /ENCODER_B: track 0.00 -> 74.0 mm, vias 0 -> 2
- net /BATTERY: track 0.00 -> 67.5 mm, vias 0 -> 2
- net /SPI_MISO: track 0.00 -> 67.1 mm, vias 0 -> 2
- net /BUTTON_LEFT: track 0.00 -> 62.0 mm
- net /BUTTON_BACK: track 0.00 -> 62.0 mm, vias 0 -> 1
- net /MCU_RESET: track 0.00 -> 59.6 mm, vias 0 -> 3
- net /SYSTEM: track 0.00 -> 53.1 mm, vias 0 -> 2
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- added copper zone on In1.Cu, net /GND
- added copper zone on In2.Cu, net /GND
Other:
- outline, holes or cut-outs redrawn
- board text added: "A1 ROUTED PROTOTYPE - PHYSICAL TESTS NOT RUN"
- board text added: "LM19-LSI OPTICAL CENTER"
- board text removed: "OPTICAL CUTOUT: VERIFY FIG.4 + LENS"
- board text removed: "PLACEMENT DRAFT - NOT FOR FABRICATION"
