File: hardware/mouse/mouse.kicad_sch (KiCad schematic)
At the start: 51 parts, among them J1 USB-C HRO TYPE-C-31-M-12, J10 Encoder: A / GND / B, J2 SWD: VDD / SWDIO / SWDCLK / G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, J3 Protected 1S 300mAh + 10k NTC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, J4 Charger status: GND / PGOOD /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, J5 BUTTON_LEFT contact, J6 BUTTON_RIGHT contact, J7 BUTTON_MIDDLE contact, J8 BUTTON_BACK contact, J9 BUTTON_FORWARD contact, SW1 PAIR TL3342, SW2 RESET TL3342, SW3 Power PCM12, U1 MDBT50Q-1MV2, U2 USBLC6-2SC6, U3 TLV70030DDCR, U4 PAW3395DM-T6QU, U5 TLV70019DDCR, U6 BQ24072RGTR, Y1 32.768kHz 12.5pF ABS07

Commit message: Route A1 prototype boards and build native firmware; bench validation pending
Parts:
- U6: footprint OpenMice:VQFN-16-1EP_3x3mm_P0.5mm_EP1.45x1.45mm -> OpenMice:BQ24072_RGT0016C
Connections:
- no-connect marks 43 -> 40
Other:
- title: mouse - electrical connectivity draft -> mouse - PAW3395 wireless prototype
- moved on the sheet: C1, C10, C11, C12, C13, C14, C15, C16, C17, C18, C19, C2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
