File: hardware/receiver/receiver.kicad_sch (KiCad schematic)
At the start: 18 parts, among them J1 USB-C HRO TYPE-C-31-M-12, J2 SWD: VDD / SWDIO / SWDCLK / G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, SW1 PAIR TL3342, SW2 RESET TL3342, U1 MDBT50Q-1MV2, U2 USBLC6-2SC6, U3 TLV70030DDCR, Y1 32.768kHz 12.5pF ABS07

Commit message: Route A1 prototype boards and build native firmware; bench validation pending
Connections:
- no-connect marks 49 -> 48
Other:
- title: receiver - electrical connectivity draft -> receiver - PAW3395 wireless prototype
- moved on the sheet: C1, C2, C3, C4, C5, C6, C7, J2, R1, R2, R3, SW1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
